Commit message: analysis part is fixed

File: Leo_sct/leo_common-ros2/leo_description/urdf/macros.xacro (robot description, xacro)
@@ -266,5 +266,5 @@
       <parent link="${link_prefix}base_link"/>
       <child link="${link_prefix}realsense_link"/>
-      <origin xyz="0.1 0 0.03" rpy="0 -0.3 0"/>
+      <origin xyz="0.1 0 0.03" rpy="0 -0.2 0"/>
     </joint>
   </xacro:macro>
@@ -454,6 +454,6 @@
           </distortion>
           <image>
-            <width>64</width>
-            <height>48</height>
+            <width>128</width>
+            <height>72</height>
             <format>R8G8B8</format>
           </image>
@@ -532,5 +532,5 @@
       <sensor name="contact_sensor" type="contact">
         <always_on>true</always_on>
-        <update_rate>100</update_rate>
+        <update_rate>20</update_rate>
         <contact>
           <collision>${link_prefix}base_footprint_fixed_joint_lump__base_collision_collision</collision>
